Commit message: convert mesh to shapes in xacro file

File: crane_x7_description/urdf/crane_x7_arm.xacro (robot description, xacro)
@@ -164,17 +164,23 @@
     <link name="${name}_link">
       <visual>
-        <origin xyz="0 0 0" rpy="0 0 0"/>
-        <geometry>
-          <mesh filename="package://crane_x7_description/meshes/visual/base_fixed_part.stl"
-              scale="1 1 1"/>
-        </geometry>
+        <origin xyz="0 0 0.0275" rpy="0 0 0"/>
+        <geometry>
+          <cylinder length="0.055" radius="0.05" />
+        </geometry>
+        <!-- <geometry>                                                                          -->
+        <!--   <mesh filename="package://crane_x7_description/meshes/visual/base_fixed_part.stl" -->
+        <!--       scale="1 1 1"/>                                                               -->
+        <!-- </geometry>                                                                         -->
         <material name="${color}"/>
       </visual>
       <collision>
-        <origin xyz="0 0 0" rpy="0 0 0"/>
-        <geometry>
-          <mesh filename="package://crane_x7_description/meshes/collision/base_fixed_part.stl"
-              scale="1 1 1"/>
-        </geometry>
+        <origin xyz="0 0 0.0275" rpy="0 0 0"/>
+        <geometry>
+          <cylinder length="0.055" radius="0.05" />
+        </geometry>
+        <!-- <geometry>                                                                             -->
+        <!--   <mesh filename="package://crane_x7_description/meshes/collision/base_fixed_part.stl" -->
+        <!--       scale="1 1 1"/>                                                                  -->
+        <!-- </geometry>                                                                            -->
       </collision>
       <inertial>
@@ -201,17 +207,23 @@
     <link name="${name}_link">
       <visual>
-        <origin xyz="0 0 0" rpy="0 0 ${M_PI}"/>
-        <geometry>
-          <mesh filename="package://crane_x7_description/meshes/visual/base_revolute_part.stl"
-              scale="1 1 1"/>
-        </geometry>
+        <origin xyz="0 0 0.06" rpy="${M_PI/2} 0 ${M_PI}"/>
+        <geometry>
+          <cylinder length="0.045" radius="0.03" />
+        </geometry>
+        <!-- <geometry>                                                                             -->
+        <!--   <mesh filename="package://crane_x7_description/meshes/visual/base_revolute_part.stl" -->
+        <!--       scale="1 1 1"/>                                                                  -->
+        <!-- </geometry>                                                                            -->
         <material name="${color}"/>
       </visual>
       <collision>
-        <origin xyz="0 0 0" rpy="0 0 ${M_PI}"/>
-        <geometry>
-          <mesh filename="package://crane_x7_description/meshes/collision/base_revolute_part.stl"
-              scale="1 1 1"/>
-        </geometry>
+        <origin xyz="0 0 0.06" rpy="${M_PI/2} 0 ${M_PI}"/>
+        <geometry>
+          <cylinder length="0.045" radius="0.03" />
+        </geometry>
+        <!-- <geometry>                                                                                -->
+        <!--   <mesh filename="package://crane_x7_description/meshes/collision/base_revolute_part.stl" -->
+        <!--       scale="1 1 1"/>                                                                     -->
+        <!-- </geometry>                                                                               -->
       </collision>
       <inertial>
@@ -238,17 +250,23 @@
     <link name="${name}_link">
       <visual>
-        <origin xyz="0 0 0" rpy="${M_PI/2} 0 0"/>
-        <geometry>
-          <mesh filename="package://crane_x7_description/meshes/visual/rotating_link_type_1_fixed_part.stl"
-              scale="1 1 1"/>
-        </geometry>
+        <origin xyz="0 0 0.04" rpy="0 0 0"/>
+        <geometry>
+          <box size="0.06 0.06 0.02" />
+        </geometry>
+        <!-- <geometry>                                                                                          -->
+        <!--   <mesh filename="package://crane_x7_description/meshes/visual/rotating_link_type_1_fixed_part.stl" -->
+        <!--       scale="1 1 1"/>                                                                               -->
+        <!-- </geometry>                                                                                         -->
         <material name="${color}"/>
       </visual>
       <collision>
-        <origin xyz="0 0 0" rpy="${M_PI/2} 0 0"/>
-        <geometry>
-          <mesh filename="package://crane_x7_description/meshes/collision/rotating_link_type_1_fixed_part.stl"
-              scale="1 1 1"/>
-        </geometry>
+        <origin xyz="0 0 0.04" rpy="0 0 0"/>
+        <geometry>
+          <box size="0.06 0.06 0.02" />
+        </geometry>
+        <!-- <geometry>                                                                                             -->
+        <!--   <mesh filename="package://crane_x7_description/meshes/collision/rotating_link_type_1_fixed_part.stl" -->
+        <!--       scale="1 1 1"/>                                                                                  -->
+        <!-- </geometry>                                                                                            -->
       </collision>
       <inertial>
@@ -266,7 +284,10 @@
         <origin xyz="0 0 0" rpy="-${M_PI/2} 0 0"/>
         <geometry>
-          <mesh filename="package://crane_x7_description/meshes/visual/joint_cover.stl"
-              scale="1 1 1"/>
-        </geometry>
+          <cylinder length="0.005" radius="0.02" />
+        </geometry>
+        <!-- <geometry>                                                                      -->
+        <!--   <mesh filename="package://crane_x7_description/meshes/visual/joint_cover.stl" -->
+        <!--       scale="1 1 1"/>                                                           -->
+        <!-- </geometry>                                                                     -->
         <material name="${joint_cover_color}"/>
       </visual>
@@ -274,7 +295,10 @@
         <origin xyz="0 0 0" rpy="-${M_PI/2} 0 0"/>
         <geometry>
-          <mesh filename="package://crane_x7_description/meshes/collision/joint_cover.stl"
-              scale="1 1 1"/>
-        </geometry>
+          <cylinder length="0.005" radius="0.02" />
+        </geometry>
+        <!-- <geometry>                                                                         -->
+        <!--   <mesh filename="package://crane_x7_description/meshes/collision/joint_cover.stl" -->
+        <!--       scale="1 1 1"/>                                                              -->
+        <!-- </geometry>                                                                        -->
       </collision>
       <inertial>
@@ -295,7 +319,10 @@
         <origin xyz="0 0 0" rpy="${M_PI/2} 0 0"/>
         <geometry>
-          <mesh filename="package://crane_x7_description/meshes/visual/joint_cover.stl"
-              scale="1 1 1"/>
-        </geometry>
+          <cylinder length="0.005" radius="0.02" />
+        </geometry>
+        <!-- <geometry>                                                                      -->
+        <!--   <mesh filename="package://crane_x7_description/meshes/visual/joint_cover.stl" -->
+        <!--       scale="1 1 1"/>                                                           -->
+        <!-- </geometry>                                                                     -->
         <material name="${joint_cover_color}"/>
       </visual>
@@ -303,7 +330,10 @@
         <origin xyz="0 0 0" rpy="${M_PI/2} 0 0"/>
         <geometry>
-          <mesh filename="package://crane_x7_description/meshes/collision/joint_cover.stl"
-              scale="1 1 1"/>
-        </geometry>
+          <cylinder length="0.005" radius="0.02" />
+        </geometry>
+        <!-- <geometry>                                                                         -->
+        <!--   <mesh filename="package://crane_x7_description/meshes/collision/joint_cover.stl" -->
+        <!--       scale="1 1 1"/>                                                              -->
+        <!-- </geometry>                                                                        -->
       </collision>
       <inertial>
@@ -339,17 +369,23 @@
     <link name="${name}_link">
       <visual>
-        <origin xyz="0 0 0" rpy="0 0 0"/>
-        <geometry>
-          <mesh filename="package://crane_x7_description/meshes/visual/rotating_link_type_1_revolute_part.stl"
-              scale="1 1 1"/>
-        </geometry>
+        <origin xyz="0 0 0.08" rpy="0 0 0"/>
+        <geometry>
+          <cylinder length="0.18" radius="0.03" />
+        </geometry>
+        <!-- <geometry>                                                                                             -->
+        <!--   <mesh filename="package://crane_x7_description/meshes/visual/rotating_link_type_1_revolute_part.stl" -->
+        <!--       scale="1 1 1"/>                                                                                  -->
+        <!-- </geometry>                                                                                            -->
         <material name="${color}"/>
       </visual>
       <collision>
-        <origin xyz="0 0 0" rpy="0 0 0"/>
-        <geometry>
-          <mesh filename="package://crane_x7_description/meshes/collision/rotating_link_type_1_revolute_part.stl"
-              scale="1 1 1"/>
-        </geometry>
+        <origin xyz="0 0 0.08" rpy="0 0 0"/>
+        <geometry>
+          <cylinder length="0.18" radius="0.03" />
+        </geometry>
+        <!-- <geometry>                                                                                                -->
+        <!--   <mesh filename="package://crane_x7_description/meshes/collision/rotating_link_type_1_revolute_part.stl" -->
+        <!--       scale="1 1 1"/>                                                                                     -->
+        <!-- </geometry>                                                                                               -->
       </collision>
       <inertial>
@@ -379,17 +415,23 @@
     <link name="${name}_link">
       <visual>
-        <origin xyz="0 0 0" rpy="${M_PI/2} 0 0"/>
-        <geometry>
-          <mesh filename="package://crane_x7_description/meshes/visual/rotating_link_type_2_fixed_part.stl"
-              scale="1 1 1"/>
-        </geometry>
+        <origin xyz="0 0 0.07" rpy="0 0 0"/>
+        <geometry>
+          <box size="0.05 0.05 0.12" />
+        </geometry>
+        <!-- <geometry>                                                                                          -->
+        <!--   <mesh filename="package://crane_x7_description/meshes/visual/rotating_link_type_2_fixed_part.stl" -->
+        <!--       scale="1 1 1"/>                                                                               -->
+        <!-- </geometry>                                                                                         -->
         <material name="${color}"/>
       </visual>
       <collision>
-        <origin xyz="0 0 0" rpy="${M_PI/2} 0 0"/>
-        <geometry>
-          <mesh filename="package://crane_x7_description/meshes/collision/rotating_link_type_2_fixed_part.stl"
-              scale="1 1 1"/>
-        </geometry>
+        <origin xyz="0 0 0.07" rpy="0 0 0"/>
+        <geometry>
+          <box size="0.05 0.05 0.12" />
+        </geometry>
+        <!-- <geometry>                                                                                             -->
+        <!--   <mesh filename="package://crane_x7_description/meshes/collision/rotating_link_type_2_fixed_part.stl" -->
+        <!--       scale="1 1 1"/>                                                                                  -->
+        <!-- </geometry>                                                                                            -->
       </collision>
       <inertial>
@@ -414,7 +456,10 @@
         <origin xyz="0 0 0" rpy="-${M_PI/2} 0 0"/>
         <geometry>
-          <mesh filename="package://crane_x7_description/meshes/visual/joint_cover.stl"
-              scale="1 1 1"/>
-        </geometry>
+          <cylinder length="0.005" radius="0.02" />
+        </geometry>
+        <!-- <geometry>                                                                      -->
+        <!--   <mesh filename="package://crane_x7_description/meshes/visual/joint_cover.stl" -->
+        <!--       scale="1 1 1"/>                                                           -->
+        <!-- </geometry>                                                                     -->
         <material name="${joint_cover_color}"/>
       </visual>
@@ -422,7 +467,10 @@
         <origin xyz="0 0 0" rpy="-${M_PI/2} 0 0"/>
         <geometry>
-          <mesh filename="package://crane_x7_description/meshes/collision/joint_cover.stl"
-              scale="1 1 1"/>
-        </geometry>
+          <cylinder length="0.005" radius="0.02" />
+        </geometry>
+        <!-- <geometry>                                                                         -->
+        <!--   <mesh filename="package://crane_x7_description/meshes/collision/joint_cover.stl" -->
+        <!--       scale="1 1 1"/>                                                              -->
+        <!-- </geometry>                                                                        -->
       </collision>
       <inertial>
@@ -443,7 +491,10 @@
         <origin xyz="0 0 0" rpy="${M_PI/2} 0 0"/>
         <geometry>
-          <mesh filename="package://crane_x7_description/meshes/visual/joint_cover.stl"
-              scale="1 1 1"/>
-        </geometry>
+          <cylinder length="0.005" radius="0.02" />
+        </geometry>
+        <!-- <geometry>                                                                      -->
+        <!--   <mesh filename="package://crane_x7_description/meshes/visual/joint_cover.stl" -->
+        <!--       scale="1 1 1"/>                                                           -->
+        <!-- </geometry>                                                                     -->
         <material name="${joint_cover_color}"/>
       </visual>
@@ -451,7 +502,10 @@
         <origin xyz="0 0 0" rpy="${M_PI/2} 0 0"/>
         <geometry>
-          <mesh filename="package://crane_x7_description/meshes/collision/joint_cover.stl"
-              scale="1 1 1"/>
-        </geometry>
+          <cylinder length="0.005" radius="0.02" />
+        </geometry>
+        <!-- <geometry>                                                                         -->
+        <!--   <mesh filename="package://crane_x7_description/meshes/collision/joint_cover.stl" -->
+        <!--       scale="1 1 1"/>                                                              -->
+        <!-- </geometry>                                                                        -->
       </collision>
       <inertial>
@@ -475,17 +529,23 @@
     <link name="${name}_link">
       <visual>
-        <origin xyz="0 0 0" rpy="0 0 0"/>
-        <geometry>
-          <mesh filename="package://crane_x7_description/meshes/visual/rotating_link_type_2_revolute_part.stl"
-              scale="1 1 1"/>
-        </geometry>
+        <origin xyz="0 0 0.05" rpy="0 0 0"/>
+        <geometry>
+          <cylinder length="0.07" radius="0.03" />
+        </geometry>
+        <!-- <geometry>                                                                                             -->
+        <!--   <mesh filename="package://crane_x7_description/meshes/visual/rotating_link_type_2_revolute_part.stl" -->
+        <!--       scale="1 1 1"/>                                                                                  -->
+        <!-- </geometry>                                                                                            -->
         <material name="${color}"/>
       </visual>
       <collision>
-        <origin xyz="0 0 0" rpy="0 0 0"/>
-        <geometry>
-          <mesh filename="package://crane_x7_description/meshes/collision/rotating_link_type_2_revolute_part.stl"
-              scale="1 1 1"/>
-        </geometry>
+        <origin xyz="0 0 0.05" rpy="0 0 0"/>
+        <geometry>
+          <cylinder length="0.07" radius="0.03" />
+        </geometry>
+        <!-- <geometry>                                                                                                -->
+        <!--   <mesh filename="package://crane_x7_description/meshes/collision/rotating_link_type_2_revolute_part.stl" -->
+        <!--       scale="1 1 1"/>                                                                                     -->
+        <!-- </geometry>                                                                                               -->
       </collision>
       <inertial>
@@ -517,7 +577,10 @@
         <origin xyz="0 0 0" rpy="${M_PI/2} 0 0"/>
         <geometry>
-          <mesh filename="package://crane_x7_description/meshes/visual/wrist.stl"
-              scale="1 1 1"/>
-        </geometry>
+          <cylinder length="0.035" radius="0.025" />
+        </geometry>
+        <!-- <geometry>                                                                -->
+        <!--   <mesh filename="package://crane_x7_description/meshes/visual/wrist.stl" -->
+        <!--       scale="1 1 1"/>                                                     -->
+        <!-- </geometry>                                                               -->
         <material name="${color}"/>
       </visual>
@@ -525,7 +588,10 @@
         <origin xyz="0 0 0" rpy="${M_PI/2} 0 0"/>
         <geometry>
-          <mesh filename="package://crane_x7_description/meshes/collision/wrist.stl"
-              scale="1 1 1"/>
-        </geometry>
+          <cylinder length="0.035" radius="0.025" />
+        </geometry>
+        <!-- <geometry>                                                                   -->
+        <!--   <mesh filename="package://crane_x7_description/meshes/collision/wrist.stl" -->
+        <!--       scale="1 1 1"/>                                                        -->
+        <!-- </geometry>                                                                  -->
       </collision>
       <inertial>

File: crane_x7_description/urdf/crane_x7_mounting_plate.xacro (robot description, xacro)
@@ -13,17 +13,23 @@
     <link name="${name}_link">
       <visual>
-        <origin xyz="0 0 0" rpy="0 0 0"/>
+        <origin xyz="0 0 0.0025" rpy="0 0 0"/>
         <geometry>
-          <mesh filename="package://crane_x7_description/meshes/visual/mounting_plate.stl"
-              scale="1 1 1"/>
+          <cylinder length="0.005" radius="0.05" />
         </geometry>
+        <!-- <geometry>                                                                         -->
+        <!--   <mesh filename="package://crane_x7_description/meshes/visual/mounting_plate.stl" -->
+        <!--       scale="1 1 1"/>                                                              -->
+        <!-- </geometry>                                                                        -->
         <material name="${color}"/>
       </visual>
       <collision>
-        <origin xyz="0 0 0" rpy="0 0 0"/>
+        <origin xyz="0 0 0.0025" rpy="0 0 0"/>
         <geometry>
-          <mesh filename="package://crane_x7_description/meshes/collision/mounting_plate.stl"
-              scale="1 1 1"/>
+          <cylinder length="0.005" radius="0.05" />
         </geometry>
+        <!-- <geometry>                                                                            -->
+        <!--   <mesh filename="package://crane_x7_description/meshes/collision/mounting_plate.stl" -->
+        <!--       scale="1 1 1"/>                                                                 -->
+        <!-- </geometry>                                                                           -->
       </collision>
       <inertial>
