Commit message: convert mesh to shapes in xacro file

File: crane_x7_description/urdf/crane_x7_rt_logos.xacro (robot description, xacro)
@@ -7,7 +7,10 @@
         <origin xyz="0 0 0" rpy="-${M_PI/2} ${M_PI/2} 0"/>
         <geometry>
-          <mesh filename="package://crane_x7_description/meshes/visual/rtcorp_logo_name.stl"
-              scale="1 1 1"/>
+          <box size="0.06 0.02 0.001" />
         </geometry>
+        <!-- <geometry>                                                                           -->
+        <!--   <mesh filename="package://crane_x7_description/meshes/visual/rtcorp_logo_name.stl" -->
+        <!--       scale="1 1 1"/>                                                                -->
+        <!-- </geometry>                                                                          -->
         <material name="logo_red">
           <color rgba="1.0 0.3 0.3 1.0"/>
@@ -32,7 +35,10 @@
         <origin xyz="0 0 0" rpy="-${M_PI/2} ${M_PI/2} 0"/>
         <geometry>
-          <mesh filename="package://crane_x7_description/meshes/visual/rtcorp_logo_rabbit.stl"
-              scale="1 1 1"/>
+          <box size="0.01 0.02 0.001" />
         </geometry>
+        <!-- <geometry>                                                                             -->
+        <!--   <mesh filename="package://crane_x7_description/meshes/visual/rtcorp_logo_rabbit.stl" -->
+        <!--       scale="1 1 1"/>                                                                  -->
+        <!-- </geometry>                                                                            -->
         <material name="logo_red"/>
       </visual>
@@ -55,7 +61,10 @@
         <origin xyz="0 0 0" rpy="${M_PI/2} -${M_PI/2} 0"/>
         <geometry>
-          <mesh filename="package://crane_x7_description/meshes/visual/rtcorp_logo_name.stl"
-              scale="1 1 1"/>
+          <box size="0.06 0.02 0.001" />
         </geometry>
+        <!-- <geometry>                                                                           -->
+        <!--   <mesh filename="package://crane_x7_description/meshes/visual/rtcorp_logo_name.stl" -->
+        <!--       scale="1 1 1"/>                                                                -->
+        <!-- </geometry>                                                                          -->
         <material name="logo_red"/>
       </visual>
@@ -78,7 +87,10 @@
         <origin xyz="0 0 0" rpy="${M_PI/2} -${M_PI/2} 0"/>
         <geometry>
-          <mesh filename="package://crane_x7_description/meshes/visual/rtcorp_logo_rabbit.stl"
-              scale="1 1 1"/>
+          <box size="0.01 0.02 0.001" />
         </geometry>
+        <!-- <geometry>                                                                             -->
+        <!--   <mesh filename="package://crane_x7_description/meshes/visual/rtcorp_logo_rabbit.stl" -->
+        <!--       scale="1 1 1"/>                                                                  -->
+        <!-- </geometry>                                                                            -->
         <material name="logo_red"/>
       </visual>

File: crane_x7_description/urdf/crane_x7_wide_two_finger_gripper.xacro (robot description, xacro)
@@ -8,17 +8,23 @@
     <link name="${name}_base_link">
       <visual>
-        <origin xyz="0 0 0" rpy="0 0 0"/>
+        <origin xyz="0 0 0.01" rpy="0 0 0"/>
         <geometry>
-          <mesh filename="package://crane_x7_description/meshes/visual/wide_two_finger_gripper_actuator.stl"
-              scale="1 1 1"/>
+          <cylinder length="0.005" radius="0.03" />
         </geometry>
+        <!-- <geometry>                                                                                           -->
+        <!--   <mesh filename="package://crane_x7_description/meshes/visual/wide_two_finger_gripper_actuator.stl" -->
+        <!--       scale="1 1 1"/>                                                                                -->
+        <!-- </geometry>                                                                                          -->
         <material name="${color}"/>
       </visual>
       <collision>
-        <origin xyz="0 0 0" rpy="0 0 0"/>
+        <origin xyz="0 0 0.01" rpy="0 0 0"/>
         <geometry>
-          <mesh filename="package://crane_x7_description/meshes/collision/wide_two_finger_gripper_actuator.stl"
-              scale="1 1 1"/>
+          <cylinder length="0.005" radius="0.03" />
         </geometry>
+        <!-- <geometry>                                                                                              -->
+        <!--   <mesh filename="package://crane_x7_description/meshes/collision/wide_two_finger_gripper_actuator.stl" -->
+        <!--       scale="1 1 1"/>                                                                                   -->
+        <!-- </geometry>                                                                                             -->
       </collision>
       <inertial>
@@ -39,17 +45,23 @@
     <link name="${name}_finger_a_link">
       <visual>
-        <origin xyz="0 0 0" rpy="${M_PI/2} 0 0"/>
+        <origin xyz="0 0 0.03" rpy="${M_PI/2} 0 0"/>
         <geometry>
-          <mesh filename="package://crane_x7_description/meshes/visual/wide_two_finger_gripper_finger_a.stl"
-              scale="1 1 1"/>
+          <box size="0.02 0.07 0.05" />
         </geometry>
+        <!-- <geometry>                                                                                           -->
+        <!--   <mesh filename="package://crane_x7_description/meshes/visual/wide_two_finger_gripper_finger_a.stl" -->
+        <!--       scale="1 1 1"/>                                                                                -->
+        <!-- </geometry>                                                                                          -->
         <material name="${color}"/>
       </visual>
       <collision>
-        <origin xyz="0 0 0" rpy="${M_PI/2} 0 0"/>
+        <origin xyz="0 0 0.03" rpy="${M_PI/2} 0 0"/>
         <geometry>
-          <mesh filename="package://crane_x7_description/meshes/collision/wide_two_finger_gripper_finger_a.stl"
-              scale="1 1 1"/>
+          <box size="0.02 0.07 0.05" />
         </geometry>
+        <!-- <geometry>                                                                                              -->
+        <!--   <mesh filename="package://crane_x7_description/meshes/collision/wide_two_finger_gripper_finger_a.stl" -->
+        <!--       scale="1 1 1"/>                                                                                   -->
+        <!-- </geometry>                                                                                             -->
       </collision>
       <inertial>
@@ -71,17 +83,23 @@
     <link name="${name}_finger_b_link">
       <visual>
-        <origin xyz="0 0 0" rpy="${M_PI/2} 0 0"/>
+        <origin xyz="0 0 0.03" rpy="${M_PI/2} 0 0"/>
         <geometry>
-          <mesh filename="package://crane_x7_description/meshes/visual/wide_two_finger_gripper_finger_b.stl"
-              scale="1 1 1"/>
+          <box size="0.02 0.07 0.05" />
         </geometry>
+        <!-- <geometry>                                                                                           -->
+        <!--   <mesh filename="package://crane_x7_description/meshes/visual/wide_two_finger_gripper_finger_b.stl" -->
+        <!--       scale="1 1 1"/>                                                                                -->
+        <!-- </geometry>                                                                                          -->
         <material name="${color}"/>
       </visual>
       <collision>
-        <origin xyz="0 0 0" rpy="${M_PI/2} 0 0"/>
+        <origin xyz="0 0 0.03" rpy="${M_PI/2} 0 0"/>
         <geometry>
-          <mesh filename="package://crane_x7_description/meshes/collision/wide_two_finger_gripper_finger_b.stl"
-              scale="1 1 1"/>
+          <box size="0.02 0.07 0.05" />
         </geometry>
+        <!-- <geometry>                                                                                              -->
+        <!--   <mesh filename="package://crane_x7_description/meshes/collision/wide_two_finger_gripper_finger_b.stl" -->
+        <!--       scale="1 1 1"/>                                                                                   -->
+        <!-- </geometry>                                                                                             -->
       </collision>
       <inertial>
