Commit message: comment out collision tags

File: crane_x7_description/urdf/crane_x7_arm.xacro (robot description, xacro)
@@ -174,14 +174,14 @@
         <material name="${color}"/>
       </visual>
-      <collision>
-        <origin xyz="0 0 0.0275" rpy="0 0 0"/>
-        <geometry>
-          <cylinder length="0.055" radius="0.05" />
-        </geometry>
-        <!-- <geometry>                                                                             -->
-        <!--   <mesh filename="package://crane_x7_description/meshes/collision/base_fixed_part.stl" -->
-        <!--       scale="1 1 1"/>                                                                  -->
-        <!-- </geometry>                                                                            -->
-      </collision>
+      <!-- <collision>                                                                                       -->
+      <!--   <origin xyz="0 0 0.0275" rpy="0 0 0"/>                                                          -->
+      <!--   <geometry>                                                                                      -->
+      <!--     <cylinder length="0.055" radius="0.05" />                                                     -->
+      <!--   </geometry>                                                                                     -->
+      <!--   <!-- <geometry>                                                                             --> -->
+      <!--   <!--   <mesh filename="package://crane_x7_description/meshes/collision/base_fixed_part.stl" --> -->
+      <!--   <!--       scale="1 1 1"/>                                                                  --> -->
+      <!--   <!-- </geometry>                                                                            --> -->
+      <!-- </collision>                                                                                      -->
       <inertial>
         <mass value="0.387313"/>
@@ -217,14 +217,14 @@
         <material name="${color}"/>
       </visual>
-      <collision>
-        <origin xyz="0 0 0.06" rpy="${M_PI/2} 0 ${M_PI}"/>
-        <geometry>
-          <cylinder length="0.045" radius="0.03" />
-        </geometry>
-        <!-- <geometry>                                                                                -->
-        <!--   <mesh filename="package://crane_x7_description/meshes/collision/base_revolute_part.stl" -->
-        <!--       scale="1 1 1"/>                                                                     -->
-        <!-- </geometry>                                                                               -->
-      </collision>
+      <!-- <collision>                                                                                          -->
+      <!--   <origin xyz="0 0 0.06" rpy="${M_PI/2} 0 ${M_PI}"/>                                                 -->
+      <!--   <geometry>                                                                                         -->
+      <!--     <cylinder length="0.045" radius="0.03" />                                                        -->
+      <!--   </geometry>                                                                                        -->
+      <!--   <!-- <geometry>                                                                                --> -->
+      <!--   <!--   <mesh filename="package://crane_x7_description/meshes/collision/base_revolute_part.stl" --> -->
+      <!--   <!--       scale="1 1 1"/>                                                                     --> -->
+      <!--   <!-- </geometry>                                                                               --> -->
+      <!-- </collision>                                                                                         -->
       <inertial>
         <mass value="0.235377"/>
@@ -260,14 +260,14 @@
         <material name="${color}"/>
       </visual>
-      <collision>
-        <origin xyz="0 0 0.04" rpy="0 0 0"/>
-        <geometry>
-          <box size="0.06 0.06 0.02" />
-        </geometry>
-        <!-- <geometry>                                                                                             -->
-        <!--   <mesh filename="package://crane_x7_description/meshes/collision/rotating_link_type_1_fixed_part.stl" -->
-        <!--       scale="1 1 1"/>                                                                                  -->
-        <!-- </geometry>                                                                                            -->
-      </collision>
+      <!-- <collision>                                                                                                       -->
+      <!--   <origin xyz="0 0 0.04" rpy="0 0 0"/>                                                                            -->
+      <!--   <geometry>                                                                                                      -->
+      <!--     <box size="0.06 0.06 0.02" />                                                                                 -->
+      <!--   </geometry>                                                                                                     -->
+      <!--   <!-- <geometry>                                                                                             --> -->
+      <!--   <!--   <mesh filename="package://crane_x7_description/meshes/collision/rotating_link_type_1_fixed_part.stl" --> -->
+      <!--   <!--       scale="1 1 1"/>                                                                                  --> -->
+      <!--   <!-- </geometry>                                                                                            --> -->
+      <!-- </collision>                                                                                                      -->
       <inertial>
         <mass value="0.120005"/>
@@ -292,14 +292,14 @@
         <material name="${joint_cover_color}"/>
       </visual>
-      <collision>
-        <origin xyz="0 0 0" rpy="-${M_PI/2} 0 0"/>
-        <geometry>
-          <cylinder length="0.005" radius="0.02" />
-        </geometry>
-        <!-- <geometry>                                                                         -->
-        <!--   <mesh filename="package://crane_x7_description/meshes/collision/joint_cover.stl" -->
-        <!--       scale="1 1 1"/>                                                              -->
-        <!-- </geometry>                                                                        -->
-      </collision>
+      <!-- <collision>                                                                                   -->
+      <!--   <origin xyz="0 0 0" rpy="-${M_PI/2} 0 0"/>                                                  -->
+      <!--   <geometry>                                                                                  -->
+      <!--     <cylinder length="0.005" radius="0.02" />                                                 -->
+      <!--   </geometry>                                                                                 -->
+      <!--   <!-- <geometry>                                                                         --> -->
+      <!--   <!--   <mesh filename="package://crane_x7_description/meshes/collision/joint_cover.stl" --> -->
+      <!--   <!--       scale="1 1 1"/>                                                              --> -->
+      <!--   <!-- </geometry>                                                                        --> -->
+      <!-- </collision>                                                                                  -->
       <inertial>
         <mass value="0.005"/>
@@ -327,14 +327,14 @@
         <material name="${joint_cover_color}"/>
       </visual>
-      <collision>
-        <origin xyz="0 0 0" rpy="${M_PI/2} 0 0"/>
-        <geometry>
-          <cylinder length="0.005" radius="0.02" />
-        </geometry>
-        <!-- <geometry>                                                                         -->
-        <!--   <mesh filename="package://crane_x7_description/meshes/collision/joint_cover.stl" -->
-        <!--       scale="1 1 1"/>                                                              -->
-        <!-- </geometry>                                                                        -->
-      </collision>
+      <!-- <collision>                                                                                   -->
+      <!--   <origin xyz="0 0 0" rpy="${M_PI/2} 0 0"/>                                                   -->
+      <!--   <geometry>                                                                                  -->
+      <!--     <cylinder length="0.005" radius="0.02" />                                                 -->
+      <!--   </geometry>                                                                                 -->
+      <!--   <!-- <geometry>                                                                         --> -->
+      <!--   <!--   <mesh filename="package://crane_x7_description/meshes/collision/joint_cover.stl" --> -->
+      <!--   <!--       scale="1 1 1"/>                                                              --> -->
+      <!--   <!-- </geometry>                                                                        --> -->
+      <!-- </collision>                                                                                  -->
       <inertial>
         <mass value="0.005"/>
@@ -379,14 +379,14 @@
         <material name="${color}"/>
       </visual>
-      <collision>
-        <origin xyz="0 0 0.08" rpy="0 0 0"/>
-        <geometry>
-          <cylinder length="0.18" radius="0.03" />
-        </geometry>
-        <!-- <geometry>                                                                                                -->
-        <!--   <mesh filename="package://crane_x7_description/meshes/collision/rotating_link_type_1_revolute_part.stl" -->
-        <!--       scale="1 1 1"/>                                                                                     -->
-        <!-- </geometry>                                                                                               -->
-      </collision>
+      <!-- <collision>                                                                                                          -->
+      <!--   <origin xyz="0 0 0.08" rpy="0 0 0"/>                                                                               -->
+      <!--   <geometry>                                                                                                         -->
+      <!--     <cylinder length="0.18" radius="0.03" />                                                                         -->
+      <!--   </geometry>                                                                                                        -->
+      <!--   <!-- <geometry>                                                                                                --> -->
+      <!--   <!--   <mesh filename="package://crane_x7_description/meshes/collision/rotating_link_type_1_revolute_part.stl" --> -->
+      <!--   <!--       scale="1 1 1"/>                                                                                     --> -->
+      <!--   <!-- </geometry>                                                                                               --> -->
+      <!-- </collision>                                                                                                         -->
       <inertial>
         <mass value="0.340878"/>
@@ -425,14 +425,14 @@
         <material name="${color}"/>
       </visual>
-      <collision>
-        <origin xyz="0 0 0.07" rpy="0 0 0"/>
-        <geometry>
-          <box size="0.05 0.05 0.12" />
-        </geometry>
-        <!-- <geometry>                                                                                             -->
-        <!--   <mesh filename="package://crane_x7_description/meshes/collision/rotating_link_type_2_fixed_part.stl" -->
-        <!--       scale="1 1 1"/>                                                                                  -->
-        <!-- </geometry>                                                                                            -->
-      </collision>
+      <!-- <collision>                                                                                                       -->
+      <!--   <origin xyz="0 0 0.07" rpy="0 0 0"/>                                                                            -->
+      <!--   <geometry>                                                                                                      -->
+      <!--     <box size="0.05 0.05 0.12" />                                                                                 -->
+      <!--   </geometry>                                                                                                     -->
+      <!--   <!-- <geometry>                                                                                             --> -->
+      <!--   <!--   <mesh filename="package://crane_x7_description/meshes/collision/rotating_link_type_2_fixed_part.stl" --> -->
+      <!--   <!--       scale="1 1 1"/>                                                                                  --> -->
+      <!--   <!-- </geometry>                                                                                            --> -->
+      <!-- </collision>                                                                                                      -->
       <inertial>
         <mass value="0.230634"/>
@@ -464,14 +464,14 @@
         <material name="${joint_cover_color}"/>
       </visual>
-      <collision>
-        <origin xyz="0 0 0" rpy="-${M_PI/2} 0 0"/>
-        <geometry>
-          <cylinder length="0.005" radius="0.02" />
-        </geometry>
-        <!-- <geometry>                                                                         -->
-        <!--   <mesh filename="package://crane_x7_description/meshes/collision/joint_cover.stl" -->
-        <!--       scale="1 1 1"/>                                                              -->
-        <!-- </geometry>                                                                        -->
-      </collision>
+      <!-- <collision>                                                                                   -->
+      <!--   <origin xyz="0 0 0" rpy="-${M_PI/2} 0 0"/>                                                  -->
+      <!--   <geometry>                                                                                  -->
+      <!--     <cylinder length="0.005" radius="0.02" />                                                 -->
+      <!--   </geometry>                                                                                 -->
+      <!--   <!-- <geometry>                                                                         --> -->
+      <!--   <!--   <mesh filename="package://crane_x7_description/meshes/collision/joint_cover.stl" --> -->
+      <!--   <!--       scale="1 1 1"/>                                                              --> -->
+      <!--   <!-- </geometry>                                                                        --> -->
+      <!-- </collision>                                                                                  -->
       <inertial>
         <mass value="0.005"/>
@@ -499,14 +499,14 @@
         <material name="${joint_cover_color}"/>
       </visual>
-      <collision>
-        <origin xyz="0 0 0" rpy="${M_PI/2} 0 0"/>
-        <geometry>
-          <cylinder length="0.005" radius="0.02" />
-        </geometry>
-        <!-- <geometry>                                                                         -->
-        <!--   <mesh filename="package://crane_x7_description/meshes/collision/joint_cover.stl" -->
-        <!--       scale="1 1 1"/>                                                              -->
-        <!-- </geometry>                                                                        -->
-      </collision>
+      <!-- <collision>                                                                                   -->
+      <!--   <origin xyz="0 0 0" rpy="${M_PI/2} 0 0"/>                                                   -->
+      <!--   <geometry>                                                                                  -->
+      <!--     <cylinder length="0.005" radius="0.02" />                                                 -->
+      <!--   </geometry>                                                                                 -->
+      <!--   <!-- <geometry>                                                                         --> -->
+      <!--   <!--   <mesh filename="package://crane_x7_description/meshes/collision/joint_cover.stl" --> -->
+      <!--   <!--       scale="1 1 1"/>                                                              --> -->
+      <!--   <!-- </geometry>                                                                        --> -->
+      <!-- </collision>                                                                                  -->
       <inertial>
         <mass value="0.005"/>
@@ -539,14 +539,14 @@
         <material name="${color}"/>
       </visual>
-      <collision>
-        <origin xyz="0 0 0.05" rpy="0 0 0"/>
-        <geometry>
-          <cylinder length="0.07" radius="0.03" />
-        </geometry>
-        <!-- <geometry>                                                                                                -->
-        <!--   <mesh filename="package://crane_x7_description/meshes/collision/rotating_link_type_2_revolute_part.stl" -->
-        <!--       scale="1 1 1"/>                                                                                     -->
-        <!-- </geometry>                                                                                               -->
-      </collision>
+      <!-- <collision>                                                                                                          -->
+      <!--   <origin xyz="0 0 0.05" rpy="0 0 0"/>                                                                               -->
+      <!--   <geometry>                                                                                                         -->
+      <!--     <cylinder length="0.07" radius="0.03" />                                                                         -->
+      <!--   </geometry>                                                                                                        -->
+      <!--   <!-- <geometry>                                                                                                --> -->
+      <!--   <!--   <mesh filename="package://crane_x7_description/meshes/collision/rotating_link_type_2_revolute_part.stl" --> -->
+      <!--   <!--       scale="1 1 1"/>                                                                                     --> -->
+      <!--   <!-- </geometry>                                                                                               --> -->
+      <!-- </collision>                                                                                                         -->
       <inertial>
         <mass value="0.192709"/>
@@ -585,14 +585,14 @@
         <material name="${color}"/>
       </visual>
-      <collision>
-        <origin xyz="0 0 0" rpy="${M_PI/2} 0 0"/>
-        <geometry>
-          <cylinder length="0.035" radius="0.025" />
-        </geometry>
-        <!-- <geometry>                                                                   -->
-        <!--   <mesh filename="package://crane_x7_description/meshes/collision/wrist.stl" -->
-        <!--       scale="1 1 1"/>                                                        -->
-        <!-- </geometry>                                                                  -->
-      </collision>
+      <!-- <collision>                                                                             -->
+      <!--   <origin xyz="0 0 0" rpy="${M_PI/2} 0 0"/>                                             -->
+      <!--   <geometry>                                                                            -->
+      <!--     <cylinder length="0.035" radius="0.025" />                                          -->
+      <!--   </geometry>                                                                           -->
+      <!--   <!-- <geometry>                                                                   --> -->
+      <!--   <!--   <mesh filename="package://crane_x7_description/meshes/collision/wrist.stl" --> -->
+      <!--   <!--       scale="1 1 1"/>                                                        --> -->
+      <!--   <!-- </geometry>                                                                  --> -->
+      <!-- </collision>                                                                            -->
       <inertial>
         <mass value="0.130549"/>
