Commit message: comment out collision tags

File: crane_x7_description/urdf/crane_x7_mounting_plate.xacro (robot description, xacro)
@@ -23,14 +23,14 @@
         <material name="${color}"/>
       </visual>
-      <collision>
-        <origin xyz="0 0 0.0025" rpy="0 0 0"/>
-        <geometry>
-          <cylinder length="0.005" radius="0.05" />
-        </geometry>
-        <!-- <geometry>                                                                            -->
-        <!--   <mesh filename="package://crane_x7_description/meshes/collision/mounting_plate.stl" -->
-        <!--       scale="1 1 1"/>                                                                 -->
-        <!-- </geometry>                                                                           -->
-      </collision>
+      <!-- <collision>                                                                                      -->
+      <!--   <origin xyz="0 0 0.0025" rpy="0 0 0"/>                                                         -->
+      <!--   <geometry>                                                                                     -->
+      <!--     <cylinder length="0.005" radius="0.05" />                                                    -->
+      <!--   </geometry>                                                                                    -->
+      <!--   <!-- <geometry>                                                                            --> -->
+      <!--   <!--   <mesh filename="package://crane_x7_description/meshes/collision/mounting_plate.stl" --> -->
+      <!--   <!--       scale="1 1 1"/>                                                                 --> -->
+      <!--   <!-- </geometry>                                                                           --> -->
+      <!-- </collision>                                                                                     -->
       <inertial>
         <mass value="0.001"/>

File: crane_x7_description/urdf/crane_x7_wide_two_finger_gripper.xacro (robot description, xacro)
@@ -18,14 +18,14 @@
         <material name="${color}"/>
       </visual>
-      <collision>
-        <origin xyz="0 0 0.01" rpy="0 0 0"/>
-        <geometry>
-          <cylinder length="0.005" radius="0.03" />
-        </geometry>
-        <!-- <geometry>                                                                                              -->
-        <!--   <mesh filename="package://crane_x7_description/meshes/collision/wide_two_finger_gripper_actuator.stl" -->
-        <!--       scale="1 1 1"/>                                                                                   -->
-        <!-- </geometry>                                                                                             -->
-      </collision>
+      <!-- <collision>                                                                                                        -->
+      <!--   <origin xyz="0 0 0.01" rpy="0 0 0"/>                                                                             -->
+      <!--   <geometry>                                                                                                       -->
+      <!--     <cylinder length="0.005" radius="0.03" />                                                                      -->
+      <!--   </geometry>                                                                                                      -->
+      <!--   <!-- <geometry>                                                                                              --> -->
+      <!--   <!--   <mesh filename="package://crane_x7_description/meshes/collision/wide_two_finger_gripper_actuator.stl" --> -->
+      <!--   <!--       scale="1 1 1"/>                                                                                   --> -->
+      <!--   <!-- </geometry>                                                                                             --> -->
+      <!-- </collision>                                                                                                       -->
       <inertial>
         <mass value="0.119807"/>
@@ -55,14 +55,14 @@
         <material name="${color}"/>
       </visual>
-      <collision>
-        <origin xyz="0 0 0.03" rpy="${M_PI/2} 0 0"/>
-        <geometry>
-          <box size="0.02 0.07 0.05" />
-        </geometry>
-        <!-- <geometry>                                                                                              -->
-        <!--   <mesh filename="package://crane_x7_description/meshes/collision/wide_two_finger_gripper_finger_a.stl" -->
-        <!--       scale="1 1 1"/>                                                                                   -->
-        <!-- </geometry>                                                                                             -->
-      </collision>
+      <!-- <collision>                                                                                                        -->
+      <!--   <origin xyz="0 0 0.03" rpy="${M_PI/2} 0 0"/>                                                                     -->
+      <!--   <geometry>                                                                                                       -->
+      <!--     <box size="0.02 0.07 0.05" />                                                                                  -->
+      <!--   </geometry>                                                                                                      -->
+      <!--   <!-- <geometry>                                                                                              --> -->
+      <!--   <!--   <mesh filename="package://crane_x7_description/meshes/collision/wide_two_finger_gripper_finger_a.stl" --> -->
+      <!--   <!--       scale="1 1 1"/>                                                                                   --> -->
+      <!--   <!-- </geometry>                                                                                             --> -->
+      <!-- </collision>                                                                                                       -->
       <inertial>
         <mass value="0.015617"/>
@@ -93,14 +93,14 @@
         <material name="${color}"/>
       </visual>
-      <collision>
-        <origin xyz="0 0 0.03" rpy="${M_PI/2} 0 0"/>
-        <geometry>
-          <box size="0.02 0.07 0.05" />
-        </geometry>
-        <!-- <geometry>                                                                                              -->
-        <!--   <mesh filename="package://crane_x7_description/meshes/collision/wide_two_finger_gripper_finger_b.stl" -->
-        <!--       scale="1 1 1"/>                                                                                   -->
-        <!-- </geometry>                                                                                             -->
-      </collision>
+      <!-- <collision>                                                                                                        -->
+      <!--   <origin xyz="0 0 0.03" rpy="${M_PI/2} 0 0"/>                                                                     -->
+      <!--   <geometry>                                                                                                       -->
+      <!--     <box size="0.02 0.07 0.05" />                                                                                  -->
+      <!--   </geometry>                                                                                                      -->
+      <!--   <!-- <geometry>                                                                                              --> -->
+      <!--   <!--   <mesh filename="package://crane_x7_description/meshes/collision/wide_two_finger_gripper_finger_b.stl" --> -->
+      <!--   <!--       scale="1 1 1"/>                                                                                   --> -->
+      <!--   <!-- </geometry>                                                                                             --> -->
+      <!-- </collision>                                                                                                       -->
       <inertial>
         <mass value="0.014417"/>
