Commit message: Fix comment out

File: crane_x7_description/urdf/crane_x7_arm.xacro (robot description, xacro)
@@ -179,8 +179,8 @@
       <!--     <cylinder length="0.055" radius="0.05" />                                                     -->
       <!--   </geometry>                                                                                     -->
-      <!--   <!-- <geometry>                                                                             --> -->
-      <!--   <!--   <mesh filename="package://crane_x7_description/meshes/collision/base_fixed_part.stl" --> -->
-      <!--   <!--       scale="1 1 1"/>                                                                  --> -->
-      <!--   <!-- </geometry>                                                                            --> -->
+      <!-- <geometry>                                                                             -->
+      <!--   <mesh filename="package://crane_x7_description/meshes/collision/base_fixed_part.stl" -->
+      <!--       scale="1 1 1"/>                                                                  -->
+      <!-- </geometry>                                                                            -->
       <!-- </collision>                                                                                      -->
       <inertial>
@@ -222,8 +222,8 @@
       <!--     <cylinder length="0.045" radius="0.03" />                                                        -->
       <!--   </geometry>                                                                                        -->
-      <!--   <!-- <geometry>                                                                                --> -->
-      <!--   <!--   <mesh filename="package://crane_x7_description/meshes/collision/base_revolute_part.stl" --> -->
-      <!--   <!--       scale="1 1 1"/>                                                                     --> -->
-      <!--   <!-- </geometry>                                                                               --> -->
+      <!-- <geometry>                                                                                -->
+      <!--   <mesh filename="package://crane_x7_description/meshes/collision/base_revolute_part.stl" -->
+      <!--       scale="1 1 1"/>                                                                     -->
+      <!-- </geometry>                                                                               -->
       <!-- </collision>                                                                                         -->
       <inertial>
@@ -265,8 +265,8 @@
       <!--     <box size="0.06 0.06 0.02" />                                                                                 -->
       <!--   </geometry>                                                                                                     -->
-      <!--   <!-- <geometry>                                                                                             --> -->
-      <!--   <!--   <mesh filename="package://crane_x7_description/meshes/collision/rotating_link_type_1_fixed_part.stl" --> -->
-      <!--   <!--       scale="1 1 1"/>                                                                                  --> -->
-      <!--   <!-- </geometry>                                                                                            --> -->
+      <!-- <geometry>                                                                                             -->
+      <!--   <mesh filename="package://crane_x7_description/meshes/collision/rotating_link_type_1_fixed_part.stl" -->
+      <!--       scale="1 1 1"/>                                                                                  -->
+      <!-- </geometry>                                                                                            -->
       <!-- </collision>                                                                                                      -->
       <inertial>
@@ -297,8 +297,8 @@
       <!--     <cylinder length="0.005" radius="0.02" />                                                 -->
       <!--   </geometry>                                                                                 -->
-      <!--   <!-- <geometry>                                                                         --> -->
-      <!--   <!--   <mesh filename="package://crane_x7_description/meshes/collision/joint_cover.stl" --> -->
-      <!--   <!--       scale="1 1 1"/>                                                              --> -->
-      <!--   <!-- </geometry>                                                                        --> -->
+      <!-- <geometry>                                                                         -->
+      <!--   <mesh filename="package://crane_x7_description/meshes/collision/joint_cover.stl" -->
+      <!--       scale="1 1 1"/>                                                              -->
+      <!-- </geometry>                                                                        -->
       <!-- </collision>                                                                                  -->
       <inertial>
@@ -332,8 +332,8 @@
       <!--     <cylinder length="0.005" radius="0.02" />                                                 -->
       <!--   </geometry>                                                                                 -->
-      <!--   <!-- <geometry>                                                                         --> -->
-      <!--   <!--   <mesh filename="package://crane_x7_description/meshes/collision/joint_cover.stl" --> -->
-      <!--   <!--       scale="1 1 1"/>                                                              --> -->
-      <!--   <!-- </geometry>                                                                        --> -->
+      <!-- <geometry>                                                                         -->
+      <!--   <mesh filename="package://crane_x7_description/meshes/collision/joint_cover.stl" -->
+      <!--       scale="1 1 1"/>                                                              -->
+      <!-- </geometry>                                                                        -->
       <!-- </collision>                                                                                  -->
       <inertial>
@@ -384,8 +384,8 @@
       <!--     <cylinder length="0.18" radius="0.03" />                                                                         -->
       <!--   </geometry>                                                                                                        -->
-      <!--   <!-- <geometry>                                                                                                --> -->
-      <!--   <!--   <mesh filename="package://crane_x7_description/meshes/collision/rotating_link_type_1_revolute_part.stl" --> -->
-      <!--   <!--       scale="1 1 1"/>                                                                                     --> -->
-      <!--   <!-- </geometry>                                                                                               --> -->
+      <!-- <geometry>                                                                                                -->
+      <!--   <mesh filename="package://crane_x7_description/meshes/collision/rotating_link_type_1_revolute_part.stl" -->
+      <!--       scale="1 1 1"/>                                                                                     -->
+      <!-- </geometry>                                                                                               -->
       <!-- </collision>                                                                                                         -->
       <inertial>
@@ -430,8 +430,8 @@
       <!--     <box size="0.05 0.05 0.12" />                                                                                 -->
       <!--   </geometry>                                                                                                     -->
-      <!--   <!-- <geometry>                                                                                             --> -->
-      <!--   <!--   <mesh filename="package://crane_x7_description/meshes/collision/rotating_link_type_2_fixed_part.stl" --> -->
-      <!--   <!--       scale="1 1 1"/>                                                                                  --> -->
-      <!--   <!-- </geometry>                                                                                            --> -->
+      <!-- <geometry>                                                                                             -->
+      <!--   <mesh filename="package://crane_x7_description/meshes/collision/rotating_link_type_2_fixed_part.stl" -->
+      <!--       scale="1 1 1"/>                                                                                  -->
+      <!-- </geometry>                                                                                            -->
       <!-- </collision>                                                                                                      -->
       <inertial>
@@ -469,8 +469,8 @@
       <!--     <cylinder length="0.005" radius="0.02" />                                                 -->
       <!--   </geometry>                                                                                 -->
-      <!--   <!-- <geometry>                                                                         --> -->
-      <!--   <!--   <mesh filename="package://crane_x7_description/meshes/collision/joint_cover.stl" --> -->
-      <!--   <!--       scale="1 1 1"/>                                                              --> -->
-      <!--   <!-- </geometry>                                                                        --> -->
+      <!-- <geometry>                                                                         -->
+      <!--   <mesh filename="package://crane_x7_description/meshes/collision/joint_cover.stl" -->
+      <!--       scale="1 1 1"/>                                                              -->
+      <!-- </geometry>                                                                        -->
       <!-- </collision>                                                                                  -->
       <inertial>
@@ -504,8 +504,8 @@
       <!--     <cylinder length="0.005" radius="0.02" />                                                 -->
       <!--   </geometry>                                                                                 -->
-      <!--   <!-- <geometry>                                                                         --> -->
-      <!--   <!--   <mesh filename="package://crane_x7_description/meshes/collision/joint_cover.stl" --> -->
-      <!--   <!--       scale="1 1 1"/>                                                              --> -->
-      <!--   <!-- </geometry>                                                                        --> -->
+      <!-- <geometry>                                                                         -->
+      <!--   <mesh filename="package://crane_x7_description/meshes/collision/joint_cover.stl" -->
+      <!--       scale="1 1 1"/>                                                              -->
+      <!-- </geometry>                                                                        -->
       <!-- </collision>                                                                                  -->
       <inertial>
@@ -544,8 +544,8 @@
       <!--     <cylinder length="0.07" radius="0.03" />                                                                         -->
       <!--   </geometry>                                                                                                        -->
-      <!--   <!-- <geometry>                                                                                                --> -->
-      <!--   <!--   <mesh filename="package://crane_x7_description/meshes/collision/rotating_link_type_2_revolute_part.stl" --> -->
-      <!--   <!--       scale="1 1 1"/>                                                                                     --> -->
-      <!--   <!-- </geometry>                                                                                               --> -->
+      <!-- <geometry>                                                                                                -->
+      <!--   <mesh filename="package://crane_x7_description/meshes/collision/rotating_link_type_2_revolute_part.stl" -->
+      <!--       scale="1 1 1"/>                                                                                     -->
+      <!-- </geometry>                                                                                               -->
       <!-- </collision>                                                                                                         -->
       <inertial>
@@ -590,8 +590,8 @@
       <!--     <cylinder length="0.035" radius="0.025" />                                          -->
       <!--   </geometry>                                                                           -->
-      <!--   <!-- <geometry>                                                                   --> -->
-      <!--   <!--   <mesh filename="package://crane_x7_description/meshes/collision/wrist.stl" --> -->
-      <!--   <!--       scale="1 1 1"/>                                                        --> -->
-      <!--   <!-- </geometry>                                                                  --> -->
+      <!-- <geometry>                                                                   -->
+      <!--   <mesh filename="package://crane_x7_description/meshes/collision/wrist.stl" -->
+      <!--       scale="1 1 1"/>                                                        -->
+      <!-- </geometry>                                                                  -->
       <!-- </collision>                                                                            -->
       <inertial>

File: crane_x7_description/urdf/crane_x7_mounting_plate.xacro (robot description, xacro)
@@ -28,8 +28,8 @@
       <!--     <cylinder length="0.005" radius="0.05" />                                                    -->
       <!--   </geometry>                                                                                    -->
-      <!--   <!-- <geometry>                                                                            --> -->
-      <!--   <!--   <mesh filename="package://crane_x7_description/meshes/collision/mounting_plate.stl" --> -->
-      <!--   <!--       scale="1 1 1"/>                                                                 --> -->
-      <!--   <!-- </geometry>                                                                           --> -->
+      <!-- <geometry>                                                                            -->
+      <!--   <mesh filename="package://crane_x7_description/meshes/collision/mounting_plate.stl" -->
+      <!--       scale="1 1 1"/>                                                                 -->
+      <!-- </geometry>                                                                           -->
       <!-- </collision>                                                                                     -->
       <inertial>

File: crane_x7_description/urdf/crane_x7_wide_two_finger_gripper.xacro (robot description, xacro)
@@ -23,8 +23,8 @@
       <!--     <cylinder length="0.005" radius="0.03" />                                                                      -->
       <!--   </geometry>                                                                                                      -->
-      <!--   <!-- <geometry>                                                                                              --> -->
-      <!--   <!--   <mesh filename="package://crane_x7_description/meshes/collision/wide_two_finger_gripper_actuator.stl" --> -->
-      <!--   <!--       scale="1 1 1"/>                                                                                   --> -->
-      <!--   <!-- </geometry>                                                                                             --> -->
+      <!-- <geometry>                                                                                              -->
+      <!--   <mesh filename="package://crane_x7_description/meshes/collision/wide_two_finger_gripper_actuator.stl" -->
+      <!--       scale="1 1 1"/>                                                                                   -->
+      <!-- </geometry>                                                                                             -->
       <!-- </collision>                                                                                                       -->
       <inertial>
@@ -60,8 +60,8 @@
       <!--     <box size="0.02 0.07 0.05" />                                                                                  -->
       <!--   </geometry>                                                                                                      -->
-      <!--   <!-- <geometry>                                                                                              --> -->
-      <!--   <!--   <mesh filename="package://crane_x7_description/meshes/collision/wide_two_finger_gripper_finger_a.stl" --> -->
-      <!--   <!--       scale="1 1 1"/>                                                                                   --> -->
-      <!--   <!-- </geometry>                                                                                             --> -->
+      <!-- <geometry>                                                                                              -->
+      <!--   <mesh filename="package://crane_x7_description/meshes/collision/wide_two_finger_gripper_finger_a.stl" -->
+      <!--       scale="1 1 1"/>                                                                                   -->
+      <!-- </geometry>                                                                                             -->
       <!-- </collision>                                                                                                       -->
       <inertial>
@@ -98,8 +98,8 @@
       <!--     <box size="0.02 0.07 0.05" />                                                                                  -->
       <!--   </geometry>                                                                                                      -->
-      <!--   <!-- <geometry>                                                                                              --> -->
-      <!--   <!--   <mesh filename="package://crane_x7_description/meshes/collision/wide_two_finger_gripper_finger_b.stl" --> -->
-      <!--   <!--       scale="1 1 1"/>                                                                                   --> -->
-      <!--   <!-- </geometry>                                                                                             --> -->
+      <!-- <geometry>                                                                                              -->
+      <!--   <mesh filename="package://crane_x7_description/meshes/collision/wide_two_finger_gripper_finger_b.stl" -->
+      <!--       scale="1 1 1"/>                                                                                   -->
+      <!-- </geometry>                                                                                             -->
       <!-- </collision>                                                                                                       -->
       <inertial>
