Commit message: comment out visual tags

File: crane_x7_description/urdf/crane_x7_arm.xacro (robot description, xacro)
@@ -163,15 +163,15 @@
     <!-- Main link -->
     <link name="${name}_link">
-      <visual>
-        <origin xyz="0 0 0.0275" rpy="0 0 0"/>
-        <geometry>
-          <cylinder length="0.055" radius="0.05" />
-        </geometry>
-        <!-- <geometry>                                                                          -->
-        <!--   <mesh filename="package://crane_x7_description/meshes/visual/base_fixed_part.stl" -->
-        <!--       scale="1 1 1"/>                                                               -->
-        <!-- </geometry>                                                                         -->
-        <material name="${color}"/>
-      </visual>
+      <!-- <visual>                                                                                       -->
+      <!--   <origin xyz="0 0 0.0275" rpy="0 0 0"/>                                                       -->
+      <!--   <geometry>                                                                                   -->
+      <!--     <cylinder length="0.055" radius="0.05" />                                                  -->
+      <!--   </geometry>                                                                                  -->
+      <!-- <geometry>                                                                          -->
+      <!--   <mesh filename="package://crane_x7_description/meshes/visual/base_fixed_part.stl" -->
+      <!--       scale="1 1 1"/>                                                               -->
+      <!-- </geometry>                                                                         -->
+      <!--   <material name="${color}"/>                                                                  -->
+      <!-- </visual>                                                                                      -->
       <!-- <collision>                                                                                       -->
       <!--   <origin xyz="0 0 0.0275" rpy="0 0 0"/>                                                          -->
@@ -206,15 +206,15 @@
       params="name color vlimit llimit ulimit attached_link">
     <link name="${name}_link">
-      <visual>
-        <origin xyz="0 0 0.06" rpy="${M_PI/2} 0 ${M_PI}"/>
-        <geometry>
-          <cylinder length="0.045" radius="0.03" />
-        </geometry>
-        <!-- <geometry>                                                                             -->
-        <!--   <mesh filename="package://crane_x7_description/meshes/visual/base_revolute_part.stl" -->
-        <!--       scale="1 1 1"/>                                                                  -->
-        <!-- </geometry>                                                                            -->
-        <material name="${color}"/>
-      </visual>
+      <!-- <visual>                                                                                          -->
+      <!--   <origin xyz="0 0 0.06" rpy="${M_PI/2} 0 ${M_PI}"/>                                              -->
+      <!--   <geometry>                                                                                      -->
+      <!--     <cylinder length="0.045" radius="0.03" />                                                     -->
+      <!--   </geometry>                                                                                     -->
+      <!-- <geometry>                                                                             -->
+      <!--   <mesh filename="package://crane_x7_description/meshes/visual/base_revolute_part.stl" -->
+      <!--       scale="1 1 1"/>                                                                  -->
+      <!-- </geometry>                                                                            -->
+      <!--   <material name="${color}"/>                                                                     -->
+      <!-- </visual>                                                                                         -->
       <!-- <collision>                                                                                          -->
       <!--   <origin xyz="0 0 0.06" rpy="${M_PI/2} 0 ${M_PI}"/>                                                 -->
@@ -249,15 +249,15 @@
     params="name color joint_cover_color">
     <link name="${name}_link">
-      <visual>
-        <origin xyz="0 0 0.04" rpy="0 0 0"/>
-        <geometry>
-          <box size="0.06 0.06 0.02" />
-        </geometry>
+      <!-- <visual>                               -->
+      <!--   <origin xyz="0 0 0.04" rpy="0 0 0"/> -->
+      <!--   <geometry>                           -->
+      <!--     <box size="0.06 0.06 0.02" />      -->
+      <!--   </geometry>                          -->
         <!-- <geometry>                                                                                          -->
         <!--   <mesh filename="package://crane_x7_description/meshes/visual/rotating_link_type_1_fixed_part.stl" -->
         <!--       scale="1 1 1"/>                                                                               -->
         <!-- </geometry>                                                                                         -->
-        <material name="${color}"/>
-      </visual>
+      <!--   <material name="${color}"/> -->
+      <!-- </visual>                     -->
       <!-- <collision>                                                                                                       -->
       <!--   <origin xyz="0 0 0.04" rpy="0 0 0"/>                                                                            -->
@@ -281,15 +281,15 @@
     <!-- TODO: Once rviz fixes its multi-material display bug, move these into the parent link -->
     <link name="${name}_joint_cover_l_link">
-      <visual>
-        <origin xyz="0 0 0" rpy="-${M_PI/2} 0 0"/>
-        <geometry>
-          <cylinder length="0.005" radius="0.02" />
-        </geometry>
+      <!-- <visual>                                      -->
+      <!--   <origin xyz="0 0 0" rpy="-${M_PI/2} 0 0"/>  -->
+      <!--   <geometry>                                  -->
+      <!--     <cylinder length="0.005" radius="0.02" /> -->
+      <!--   </geometry>                                 -->
         <!-- <geometry>                                                                      -->
         <!--   <mesh filename="package://crane_x7_description/meshes/visual/joint_cover.stl" -->
         <!--       scale="1 1 1"/>                                                           -->
         <!-- </geometry>                                                                     -->
-        <material name="${joint_cover_color}"/>
-      </visual>
+      <!--   <material name="${joint_cover_color}"/> -->
+      <!-- </visual>                                 -->
       <!-- <collision>                                                                                   -->
       <!--   <origin xyz="0 0 0" rpy="-${M_PI/2} 0 0"/>                                                  -->
@@ -316,15 +316,15 @@
     </joint>
     <link name="${name}_joint_cover_r_link">
-      <visual>
-        <origin xyz="0 0 0" rpy="${M_PI/2} 0 0"/>
-        <geometry>
-          <cylinder length="0.005" radius="0.02" />
-        </geometry>
+      <!-- <visual>                                      -->
+      <!--   <origin xyz="0 0 0" rpy="${M_PI/2} 0 0"/>   -->
+      <!--   <geometry>                                  -->
+      <!--     <cylinder length="0.005" radius="0.02" /> -->
+      <!--   </geometry>                                 -->
         <!-- <geometry>                                                                      -->
         <!--   <mesh filename="package://crane_x7_description/meshes/visual/joint_cover.stl" -->
         <!--       scale="1 1 1"/>                                                           -->
         <!-- </geometry>                                                                     -->
-        <material name="${joint_cover_color}"/>
-      </visual>
+      <!--   <material name="${joint_cover_color}"/> -->
+      <!-- </visual>                                 -->
       <!-- <collision>                                                                                   -->
       <!--   <origin xyz="0 0 0" rpy="${M_PI/2} 0 0"/>                                                   -->
@@ -368,15 +368,15 @@
     </joint>
     <link name="${name}_link">
-      <visual>
-        <origin xyz="0 0 0.08" rpy="0 0 0"/>
-        <geometry>
-          <cylinder length="0.18" radius="0.03" />
-        </geometry>
+      <!-- <visual>                                     -->
+      <!--   <origin xyz="0 0 0.08" rpy="0 0 0"/>       -->
+      <!--   <geometry>                                 -->
+      <!--     <cylinder length="0.18" radius="0.03" /> -->
+      <!--   </geometry>                                -->
         <!-- <geometry>                                                                                             -->
         <!--   <mesh filename="package://crane_x7_description/meshes/visual/rotating_link_type_1_revolute_part.stl" -->
         <!--       scale="1 1 1"/>                                                                                  -->
         <!-- </geometry>                                                                                            -->
-        <material name="${color}"/>
-      </visual>
+      <!--   <material name="${color}"/> -->
+      <!-- </visual>                     -->
       <!-- <collision>                                                                                                          -->
       <!--   <origin xyz="0 0 0.08" rpy="0 0 0"/>                                                                               -->
@@ -414,15 +414,15 @@
       params="name color vlimit llimit ulimit joint_cover_color attached_link *origin">
     <link name="${name}_link">
-      <visual>
-        <origin xyz="0 0 0.07" rpy="0 0 0"/>
-        <geometry>
-          <box size="0.05 0.05 0.12" />
-        </geometry>
+      <!-- <visual>                               -->
+      <!--   <origin xyz="0 0 0.07" rpy="0 0 0"/> -->
+      <!--   <geometry>                           -->
+      <!--     <box size="0.05 0.05 0.12" />      -->
+      <!--   </geometry>                          -->
         <!-- <geometry>                                                                                          -->
         <!--   <mesh filename="package://crane_x7_description/meshes/visual/rotating_link_type_2_fixed_part.stl" -->
         <!--       scale="1 1 1"/>                                                                               -->
         <!-- </geometry>                                                                                         -->
-        <material name="${color}"/>
-      </visual>
+      <!--   <material name="${color}"/> -->
+      <!-- </visual>                     -->
       <!-- <collision>                                                                                                       -->
       <!--   <origin xyz="0 0 0.07" rpy="0 0 0"/>                                                                            -->
@@ -453,15 +453,15 @@
     <!-- TODO: Once rviz fixes its multi-material display bug, move these into the parent link -->
     <link name="${name}_joint_cover_l_link">
-      <visual>
-        <origin xyz="0 0 0" rpy="-${M_PI/2} 0 0"/>
-        <geometry>
-          <cylinder length="0.005" radius="0.02" />
-        </geometry>
+      <!-- <visual>                                      -->
+      <!--   <origin xyz="0 0 0" rpy="-${M_PI/2} 0 0"/>  -->
+      <!--   <geometry>                                  -->
+      <!--     <cylinder length="0.005" radius="0.02" /> -->
+      <!--   </geometry>                                 -->
         <!-- <geometry>                                                                      -->
         <!--   <mesh filename="package://crane_x7_description/meshes/visual/joint_cover.stl" -->
         <!--       scale="1 1 1"/>                                                           -->
         <!-- </geometry>                                                                     -->
-        <material name="${joint_cover_color}"/>
-      </visual>
+      <!--   <material name="${joint_cover_color}"/> -->
+      <!-- </visual>                                 -->
       <!-- <collision>                                                                                   -->
       <!--   <origin xyz="0 0 0" rpy="-${M_PI/2} 0 0"/>                                                  -->
@@ -488,15 +488,15 @@
     </joint>
     <link name="${name}_joint_cover_r_link">
-      <visual>
-        <origin xyz="0 0 0" rpy="${M_PI/2} 0 0"/>
-        <geometry>
-          <cylinder length="0.005" radius="0.02" />
-        </geometry>
+      <!-- <visual>                                      -->
+      <!--   <origin xyz="0 0 0" rpy="${M_PI/2} 0 0"/>   -->
+      <!--   <geometry>                                  -->
+      <!--     <cylinder length="0.005" radius="0.02" /> -->
+      <!--   </geometry>                                 -->
         <!-- <geometry>                                                                      -->
         <!--   <mesh filename="package://crane_x7_description/meshes/visual/joint_cover.stl" -->
         <!--       scale="1 1 1"/>                                                           -->
         <!-- </geometry>                                                                     -->
-        <material name="${joint_cover_color}"/>
-      </visual>
+      <!--   <material name="${joint_cover_color}"/> -->
+      <!-- </visual>                                 -->
       <!-- <collision>                                                                                   -->
       <!--   <origin xyz="0 0 0" rpy="${M_PI/2} 0 0"/>                                                   -->
@@ -528,15 +528,15 @@
       params="name color vlimit llimit ulimit attached_link logos_definition *origin">
     <link name="${name}_link">
-      <visual>
-        <origin xyz="0 0 0.05" rpy="0 0 0"/>
-        <geometry>
-          <cylinder length="0.07" radius="0.03" />
-        </geometry>
+      <!-- <visual>                                     -->
+      <!--   <origin xyz="0 0 0.05" rpy="0 0 0"/>       -->
+      <!--   <geometry>                                 -->
+      <!--     <cylinder length="0.07" radius="0.03" /> -->
+      <!--   </geometry>                                -->
         <!-- <geometry>                                                                                             -->
         <!--   <mesh filename="package://crane_x7_description/meshes/visual/rotating_link_type_2_revolute_part.stl" -->
         <!--       scale="1 1 1"/>                                                                                  -->
         <!-- </geometry>                                                                                            -->
-        <material name="${color}"/>
-      </visual>
+      <!--   <material name="${color}"/> -->
+      <!-- </visual>                     -->
       <!-- <collision>                                                                                                          -->
       <!--   <origin xyz="0 0 0.05" rpy="0 0 0"/>                                                                               -->
@@ -574,15 +574,15 @@
       params="name color vlimit llimit ulimit attached_link *origin">
     <link name="${name}_link">
-      <visual>
-        <origin xyz="0 0 0" rpy="${M_PI/2} 0 0"/>
-        <geometry>
-          <cylinder length="0.035" radius="0.025" />
-        </geometry>
+      <!-- <visual>                                       -->
+      <!--   <origin xyz="0 0 0" rpy="${M_PI/2} 0 0"/>    -->
+      <!--   <geometry>                                   -->
+      <!--     <cylinder length="0.035" radius="0.025" /> -->
+      <!--   </geometry>                                  -->
         <!-- <geometry>                                                                -->
         <!--   <mesh filename="package://crane_x7_description/meshes/visual/wrist.stl" -->
         <!--       scale="1 1 1"/>                                                     -->
         <!-- </geometry>                                                               -->
-        <material name="${color}"/>
-      </visual>
+      <!--   <material name="${color}"/> -->
+      <!-- </visual>                     -->
       <!-- <collision>                                                                             -->
       <!--   <origin xyz="0 0 0" rpy="${M_PI/2} 0 0"/>                                             -->

File: crane_x7_description/urdf/crane_x7_mounting_plate.xacro (robot description, xacro)
@@ -12,15 +12,15 @@
     </joint>
     <link name="${name}_link">
-      <visual>
-        <origin xyz="0 0 0.0025" rpy="0 0 0"/>
-        <geometry>
-          <cylinder length="0.005" radius="0.05" />
-        </geometry>
-        <!-- <geometry>                                                                         -->
-        <!--   <mesh filename="package://crane_x7_description/meshes/visual/mounting_plate.stl" -->
-        <!--       scale="1 1 1"/>                                                              -->
-        <!-- </geometry>                                                                        -->
-        <material name="${color}"/>
-      </visual>
+      <!-- <visual>                                                                                      -->
+      <!--   <origin xyz="0 0 0.0025" rpy="0 0 0"/>                                                      -->
+      <!--   <geometry>                                                                                  -->
+      <!--     <cylinder length="0.005" radius="0.05" />                                                 -->
+      <!--   </geometry>                                                                                 -->
+      <!-- <geometry>                                                                         -->
+      <!--   <mesh filename="package://crane_x7_description/meshes/visual/mounting_plate.stl" -->
+      <!--       scale="1 1 1"/>                                                              -->
+      <!-- </geometry>                                                                        -->
+      <!--   <material name="${color}"/>                                                                 -->
+      <!-- </visual>                                                                                     -->
       <!-- <collision>                                                                                      -->
       <!--   <origin xyz="0 0 0.0025" rpy="0 0 0"/>                                                         -->
