Commit message: comment out visual tags

File: crane_x7_description/urdf/crane_x7_rt_logos.xacro (robot description, xacro)
@@ -4,17 +4,17 @@
     <!-- Left side logo text -->
     <link name="${name}_logo_text_l_link">
-      <visual>
-        <origin xyz="0 0 0" rpy="-${M_PI/2} ${M_PI/2} 0"/>
-        <geometry>
-          <box size="0.06 0.02 0.001" />
-        </geometry>
+      <!-- <visual>                                             -->
+      <!--   <origin xyz="0 0 0" rpy="-${M_PI/2} ${M_PI/2} 0"/> -->
+      <!--   <geometry>                                         -->
+      <!--     <box size="0.06 0.02 0.001" />                   -->
+      <!--   </geometry>                                        -->
         <!-- <geometry>                                                                           -->
         <!--   <mesh filename="package://crane_x7_description/meshes/visual/rtcorp_logo_name.stl" -->
         <!--       scale="1 1 1"/>                                                                -->
         <!-- </geometry>                                                                          -->
-        <material name="logo_red">
-          <color rgba="1.0 0.3 0.3 1.0"/>
-        </material>
-      </visual>
+      <!--   <material name="logo_red">        -->
+      <!--     <color rgba="1.0 0.3 0.3 1.0"/> -->
+      <!--   </material>                       -->
+      <!-- </visual>                           -->
       <inertial>
         <mass value="0"/>
@@ -32,15 +32,15 @@
     <!-- Left side logo symbol -->
     <link name="${name}_logo_symbol_l_link">
-      <visual>
-        <origin xyz="0 0 0" rpy="-${M_PI/2} ${M_PI/2} 0"/>
-        <geometry>
-          <box size="0.01 0.02 0.001" />
-        </geometry>
+      <!-- <visual>                                             -->
+      <!--   <origin xyz="0 0 0" rpy="-${M_PI/2} ${M_PI/2} 0"/> -->
+      <!--   <geometry>                                         -->
+      <!--     <box size="0.01 0.02 0.001" />                   -->
+      <!--   </geometry>                                        -->
         <!-- <geometry>                                                                             -->
         <!--   <mesh filename="package://crane_x7_description/meshes/visual/rtcorp_logo_rabbit.stl" -->
         <!--       scale="1 1 1"/>                                                                  -->
         <!-- </geometry>                                                                            -->
-        <material name="logo_red"/>
-      </visual>
+      <!--   <material name="logo_red"/> -->
+      <!-- </visual>                     -->
       <inertial>
         <mass value="0"/>
@@ -58,15 +58,15 @@
     <!-- Right side logo text -->
     <link name="${name}_logo_text_r_link">
-      <visual>
-        <origin xyz="0 0 0" rpy="${M_PI/2} -${M_PI/2} 0"/>
-        <geometry>
-          <box size="0.06 0.02 0.001" />
-        </geometry>
+      <!-- <visual>                                             -->
+      <!--   <origin xyz="0 0 0" rpy="${M_PI/2} -${M_PI/2} 0"/> -->
+      <!--   <geometry>                                         -->
+      <!--     <box size="0.06 0.02 0.001" />                   -->
+      <!--   </geometry>                                        -->
         <!-- <geometry>                                                                           -->
         <!--   <mesh filename="package://crane_x7_description/meshes/visual/rtcorp_logo_name.stl" -->
         <!--       scale="1 1 1"/>                                                                -->
         <!-- </geometry>                                                                          -->
-        <material name="logo_red"/>
-      </visual>
+      <!--   <material name="logo_red"/> -->
+      <!-- </visual>                     -->
       <inertial>
         <mass value="0"/>
@@ -84,15 +84,15 @@
     <!-- Right side logo symbol -->
     <link name="${name}_logo_symbol_r_link">
-      <visual>
-        <origin xyz="0 0 0" rpy="${M_PI/2} -${M_PI/2} 0"/>
-        <geometry>
-          <box size="0.01 0.02 0.001" />
-        </geometry>
+      <!-- <visual>                                             -->
+      <!--   <origin xyz="0 0 0" rpy="${M_PI/2} -${M_PI/2} 0"/> -->
+      <!--   <geometry>                                         -->
+      <!--     <box size="0.01 0.02 0.001" />                   -->
+      <!--   </geometry>                                        -->
         <!-- <geometry>                                                                             -->
         <!--   <mesh filename="package://crane_x7_description/meshes/visual/rtcorp_logo_rabbit.stl" -->
         <!--       scale="1 1 1"/>                                                                  -->
         <!-- </geometry>                                                                            -->
-        <material name="logo_red"/>
-      </visual>
+      <!--   <material name="logo_red"/> -->
+      <!-- </visual>                     -->
       <inertial>
         <mass value="0"/>

File: crane_x7_description/urdf/crane_x7_wide_two_finger_gripper.xacro (robot description, xacro)
@@ -7,15 +7,15 @@
     params="name color vlimit">
     <link name="${name}_base_link">
-      <visual>
-        <origin xyz="0 0 0.01" rpy="0 0 0"/>
-        <geometry>
-          <cylinder length="0.005" radius="0.03" />
-        </geometry>
+      <!-- <visual>                                      -->
+      <!--   <origin xyz="0 0 0.01" rpy="0 0 0"/>        -->
+      <!--   <geometry>                                  -->
+      <!--     <cylinder length="0.005" radius="0.03" /> -->
+      <!--   </geometry>                                 -->
         <!-- <geometry>                                                                                           -->
         <!--   <mesh filename="package://crane_x7_description/meshes/visual/wide_two_finger_gripper_actuator.stl" -->
         <!--       scale="1 1 1"/>                                                                                -->
         <!-- </geometry>                                                                                          -->
-        <material name="${color}"/>
-      </visual>
+      <!--   <material name="${color}"/> -->
+      <!-- </visual>                     -->
       <!-- <collision>                                                                                                        -->
       <!--   <origin xyz="0 0 0.01" rpy="0 0 0"/>                                                                             -->
@@ -44,15 +44,15 @@
     </joint>
     <link name="${name}_finger_a_link">
-      <visual>
-        <origin xyz="0 0 0.03" rpy="${M_PI/2} 0 0"/>
-        <geometry>
-          <box size="0.02 0.07 0.05" />
-        </geometry>
+      <!-- <visual>                                       -->
+      <!--   <origin xyz="0 0 0.03" rpy="${M_PI/2} 0 0"/> -->
+      <!--   <geometry>                                   -->
+      <!--     <box size="0.02 0.07 0.05" />              -->
+      <!--   </geometry>                                  -->
         <!-- <geometry>                                                                                           -->
         <!--   <mesh filename="package://crane_x7_description/meshes/visual/wide_two_finger_gripper_finger_a.stl" -->
         <!--       scale="1 1 1"/>                                                                                -->
         <!-- </geometry>                                                                                          -->
-        <material name="${color}"/>
-      </visual>
+      <!--   <material name="${color}"/> -->
+      <!-- </visual>                     -->
       <!-- <collision>                                                                                                        -->
       <!--   <origin xyz="0 0 0.03" rpy="${M_PI/2} 0 0"/>                                                                     -->
@@ -82,15 +82,15 @@
     </joint>
     <link name="${name}_finger_b_link">
-      <visual>
-        <origin xyz="0 0 0.03" rpy="${M_PI/2} 0 0"/>
-        <geometry>
-          <box size="0.02 0.07 0.05" />
-        </geometry>
+      <!-- <visual>                                       -->
+      <!--   <origin xyz="0 0 0.03" rpy="${M_PI/2} 0 0"/> -->
+      <!--   <geometry>                                   -->
+      <!--     <box size="0.02 0.07 0.05" />              -->
+      <!--   </geometry>                                  -->
         <!-- <geometry>                                                                                           -->
         <!--   <mesh filename="package://crane_x7_description/meshes/visual/wide_two_finger_gripper_finger_b.stl" -->
         <!--       scale="1 1 1"/>                                                                                -->
         <!-- </geometry>                                                                                          -->
-        <material name="${color}"/>
-      </visual>
+      <!--   <material name="${color}"/> -->
+      <!-- </visual>                     -->
       <!-- <collision>                                                                                                        -->
       <!--   <origin xyz="0 0 0.03" rpy="${M_PI/2} 0 0"/>                                                                     -->
